File: v.2/Pneumatic/radical-pneu.brd (EAGLE design)
At the start: 30.5 x 50.8 mm, 41 parts, among them IC3 ATMEGA328, Q1 16Mhz, U2 NCP1117-5

Commit message: added 5th pin
5th pin will allow dynamic addressing of the connected boards.

also added holes in the corners for fixtures.
Parts:
- removed JP2, JP3: (no value), SparkFun-Connectors:1X04
- added R14: 10k, SparkFun-Resistors:0805
- added U$23, U$24: 1X05, digikey:1X05_TIGHT
- moved C5 1.89 mm to (4.14, 3.43), turned to 270 degrees
- moved C10 0.64 mm to (23.5, 17.7)
- moved R3 0.55 mm to (22.3, 2.16)
Connections:
- removed net D2/BTN: IC3.32
- new net D2/OUT: IC3.32, U$23.P$4
- new net IN_PORT: IC3.24, R14.2, U$24.P$4
- net GND: now also R14.1, U$23.P$5, U$24.P$5; no longer JP2.1, JP3.1
- net SCL: now also U$23.P$3, U$24.P$3; no longer JP2.3, JP3.3
- net SDA: now also U$23.P$2, U$24.P$2; no longer JP2.2, JP3.2
- net VIN: now also U$23.P$1, U$24.P$1; no longer JP2.4, JP3.4
Routing:
- net IN_PORT: track 0.00 -> 13.9 mm, vias 0 -> 3
- net D2/OUT: track 0.00 -> 7.56 mm, vias 0 -> 1
- net +5V: track 214.4 -> 218.9 mm
- net DTR: track 6.10 -> 2.21 mm
- net TX: track 43.8 -> 45.4 mm
- net D10: track 49.2 -> 50.7 mm
- net D8: track 74.7 -> 76.1 mm
- net D7: track 55.3 -> 56.6 mm
- net RX: track 103.3 -> 101.9 mm
- net D4: track 33.9 -> 34.7 mm
- net RESET: track 44.7 -> 44.0 mm
- net GND: vias 73 -> 112
Other:
- board text added: "LEFT"
- board text added: "RIGHT"
